Commit message: Update manip stack: hardware interface and bringup configs

File: src/manip_description/urdf/gripper.xacro (robot description, xacro)
@@ -67,5 +67,4 @@
     <axis xyz="0 -1 0"/>
     <limit lower="-1.0" upper="1.0" effort="1" velocity="5"/>
-    <mimic joint="joint6" offset="0"/>
     </joint>
 </robot>

File: src/manip_description/urdf/manip.ros2_control.xacro (robot description, xacro)
@@ -1,45 +1,65 @@
 <?xml version="1.0"?>
 <robot xmlns:xacro="http://www.ros.org/wiki/xacro">
-        <ros2_control name="Arm" type="system">
-            <hardware>
+    <xacro:arg name="use_mock_components" default="true"/>
+    <ros2_control name="Arm" type="system">
+        <hardware>
+            <xacro:if value="$(arg use_mock_components)">
                 <!-- By default, set up controllers for simulation. This won't work on real hardware -->
                 <plugin>mock_components/GenericSystem</plugin>
-            </hardware>
-            <joint name="joint1">
-                <command_interface name="position"/>
-                <state_interface name="position">
-                  <param name="initial_value">0.0</param>
-                </state_interface>
-            </joint>
-            <joint name="joint2">
-                <command_interface name="position"/>
-                <state_interface name="position">
-                  <param name="initial_value">0.0</param>
-                </state_interface>
-            </joint>
-            <joint name="joint3">
-                <command_interface name="position"/>
-                <state_interface name="position">
-                  <param name="initial_value">0.0</param>
-                </state_interface>
-            </joint>
-            <joint name="joint4">
-                <command_interface name="position"/>
-                <state_interface name="position">
-                  <param name="initial_value">0.0</param>
-                </state_interface>
-            </joint>
-            <joint name="joint5">
-                <command_interface name="position"/>
-                <state_interface name="position">
-                  <param name="initial_value">0.0</param>
-                </state_interface>
-            </joint>
-            <joint name="joint6">
-                <command_interface name="position"/>
-                <state_interface name="position">
-                  <param name="initial_value">0.0</param>
-                </state_interface>
-            </joint>
-        </ros2_control>
+            </xacro:if>
+            <xacro:unless value="$(arg use_mock_components)">
+                <plugin>arm_hardware/ArmHardwareInterface</plugin>
+                <param name="joint1_motor_id">1</param>
+                <param name="joint2_motor_id">2</param>
+                <param name="joint3_motor_id">3</param>
+                <param name="joint4_motor_id">4</param>
+                <param name="joint5_motor_id">5</param>
+                <param name="joint6_motor_id">6</param>
+                <param name="joint7_motor_id">7</param>
+                <param name="dynamixel_port">/dev/ttyUSB0</param>
+            </xacro:unless>
+        </hardware>
+        <joint name="joint1">
+            <command_interface name="position"/>
+            <state_interface name="position">
+                <param name="initial_value">0.0</param>
+            </state_interface>
+        </joint>
+        <joint name="joint2">
+            <command_interface name="position"/>
+            <state_interface name="position">
+                <param name="initial_value">0.0</param>
+            </state_interface>
+        </joint>
+        <joint name="joint3">
+            <command_interface name="position"/>
+            <state_interface name="position">
+                <param name="initial_value">0.0</param>
+            </state_interface>
+        </joint>
+        <joint name="joint4">
+            <command_interface name="position"/>
+            <state_interface name="position">
+                <param name="initial_value">0.0</param>
+            </state_interface>
+        </joint>
+        <joint name="joint5">
+            <command_interface name="position"/>
+            <state_interface name="position">
+                <param name="initial_value">0.0</param>
+            </state_interface>
+        </joint>
+        <joint name="joint6">
+            <command_interface name="position"/>
+            <state_interface name="position">
+                <param name="initial_value">0.0</param>
+            </state_interface>
+        </joint>
+        <joint name="joint7">
+            <command_interface name="position"/>
+            <state_interface name="position">
+                <param name="initial_value">0.0</param>
+            </state_interface>
+        </joint>
+    </ros2_control>
 </robot>

File: src/manip_moveit_config/config/manip.ros2_control.xacro (robot description, xacro)
@@ -44,4 +44,10 @@
                 </state_interface>
             </joint>
+            <joint name="joint7">
+                <command_interface name="position"/>
+                <state_interface name="position">
+                  <param name="initial_value">${initial_positions['joint7']}</param>
+                </state_interface>
+            </joint>
         </ros2_control>
     </xacro:macro>
