Commit message: Foi adicionado novas posições de mesa para as ações de place. As posições são Mesa0, Mesa0.1 e Mesa0.2.

File: src/manip_description/urdf/arm.xacro (robot description, xacro)
@@ -160,5 +160,5 @@
   </xacro:sensor_d455>
   <!-- ================= ARM JOINTS ================= -->
-  <joint name="joint1" type="revolute">
+  <joint name="manip_joint1" type="revolute">
     <parent link="base_link"/>
     <child link="link1"/>
@@ -167,5 +167,5 @@
            effort="10" velocity="1"/>
   </joint>
-  <joint name="joint2" type="revolute">
+  <joint name="manip_joint2" type="revolute">
     <parent link="link1"/>
     <child link="link2"/>
@@ -175,5 +175,5 @@
            effort="10" velocity="3"/>
   </joint>
-  <joint name="joint3" type="revolute">
+  <joint name="manip_joint3" type="revolute">
     <parent link="link2"/>
     <child link="link3"/>
@@ -183,5 +183,5 @@
            effort="10" velocity="1"/>
   </joint>
-  <joint name="joint4" type="revolute">
+  <joint name="manip_joint4" type="revolute">
     <parent link="link3"/>
     <child link="link4"/>
@@ -191,5 +191,5 @@
            effort="10" velocity="1"/>
   </joint>
-  <joint name="joint5" type="revolute">
+  <joint name="manip_joint5" type="revolute">
     <parent link="link4"/>
     <child link="link5"/>

File: src/manip_description/urdf/gripper.xacro (robot description, xacro)
@@ -34,5 +34,5 @@
     </inertial>
     </link>
-    <joint name="joint6" type="revolute">
+    <joint name="manip_joint6" type="revolute">
     <parent link="gripper_base_link"/>
     <child link="finger_left"/>
@@ -61,5 +61,5 @@
     </inertial>
     </link>
-    <joint name="joint7" type="revolute">
+    <joint name="manip_joint7" type="revolute">
     <parent link="gripper_base_link"/>
     <child link="finger_right"/>

File: src/manip_description/urdf/manip.ros2_control.xacro (robot description, xacro)
@@ -10,15 +10,15 @@
             <xacro:unless value="$(arg use_mock_components)">
                 <plugin>arm_hardware/ArmHardwareInterface</plugin>
-                <param name="joint1_motor_id">1</param>
-                <param name="joint2_motor_id">2</param>
-                <param name="joint3_motor_id">3</param>
-                <param name="joint4_motor_id">4</param>
-                <param name="joint5_motor_id">5</param>
-                <param name="joint6_motor_id">6</param>
-                <param name="joint7_motor_id">7</param>
+                <param name="manip_joint1_motor_id">1</param>
+                <param name="manip_joint2_motor_id">2</param>
+                <param name="manip_joint3_motor_id">3</param>
+                <param name="manip_joint4_motor_id">4</param>
+                <param name="manip_joint5_motor_id">5</param>
+                <param name="manip_joint6_motor_id">6</param>
+                <param name="manip_joint7_motor_id">7</param>
                 <param name="dynamixel_port">/dev/ttyUSB0</param>
             </xacro:unless>
         </hardware>
-        <joint name="joint1">
+        <joint name="manip_joint1">
             <command_interface name="position"/>
             <state_interface name="position">
@@ -26,5 +26,5 @@
             </state_interface>
         </joint>
-        <joint name="joint2">
+        <joint name="manip_joint2">
             <command_interface name="position"/>
             <state_interface name="position">
@@ -32,5 +32,5 @@
             </state_interface>
         </joint>
-        <joint name="joint3">
+        <joint name="manip_joint3">
             <command_interface name="position"/>
             <state_interface name="position">
@@ -38,5 +38,5 @@
             </state_interface>
         </joint>
-        <joint name="joint4">
+        <joint name="manip_joint4">
             <command_interface name="position"/>
             <state_interface name="position">
@@ -44,5 +44,5 @@
             </state_interface>
         </joint>
-        <joint name="joint5">
+        <joint name="manip_joint5">
             <command_interface name="position"/>
             <state_interface name="position">
@@ -50,5 +50,5 @@
             </state_interface>
         </joint>
-        <joint name="joint6">
+        <joint name="manip_joint6">
             <command_interface name="position"/>
             <state_interface name="position">
@@ -56,5 +56,5 @@
             </state_interface>
         </joint>
-        <joint name="joint7">
+        <joint name="manip_joint7">
             <command_interface name="position"/>
             <state_interface name="position">

File: src/manip_moveit_config/config/manip.ros2_control.xacro (robot description, xacro)
@@ -8,44 +8,44 @@
                 <plugin>mock_components/GenericSystem</plugin>
             </hardware>
-            <joint name="joint1">
+            <joint name="manip_joint1">
                 <command_interface name="position"/>
                 <state_interface name="position">
-                  <param name="initial_value">${initial_positions['joint1']}</param>
+                  <param name="initial_value">${initial_positions['manip_joint1']}</param>
                 </state_interface>
             </joint>
-            <joint name="joint2">
+            <joint name="manip_joint2">
                 <command_interface name="position"/>
                 <state_interface name="position">
-                  <param name="initial_value">${initial_positions['joint2']}</param>
+                  <param name="initial_value">${initial_positions['manip_joint2']}</param>
                 </state_interface>
             </joint>
-            <joint name="joint3">
+            <joint name="manip_joint3">
                 <command_interface name="position"/>
                 <state_interface name="position">
-                  <param name="initial_value">${initial_positions['joint3']}</param>
+                  <param name="initial_value">${initial_positions['manip_joint3']}</param>
                 </state_interface>
             </joint>
-            <joint name="joint4">
+            <joint name="manip_joint4">
                 <command_interface name="position"/>
                 <state_interface name="position">
-                  <param name="initial_value">${initial_positions['joint4']}</param>
+                  <param name="initial_value">${initial_positions['manip_joint4']}</param>
                 </state_interface>
             </joint>
-            <joint name="joint5">
+            <joint name="manip_joint5">
                 <command_interface name="position"/>
                 <state_interface name="position">
-                  <param name="initial_value">${initial_positions['joint5']}</param>
+                  <param name="initial_value">${initial_positions['manip_joint5']}</param>
                 </state_interface>
             </joint>
-            <joint name="joint6">
+            <joint name="manip_joint6">
                 <command_interface name="position"/>
                 <state_interface name="position">
-                  <param name="initial_value">${initial_positions['joint6']}</param>
+                  <param name="initial_value">${initial_positions['manip_joint6']}</param>
                 </state_interface>
             </joint>
-            <joint name="joint7">
+            <joint name="manip_joint7">
                 <command_interface name="position"/>
                 <state_interface name="position">
-                  <param name="initial_value">${initial_positions['joint7']}</param>
+                  <param name="initial_value">${initial_positions['manip_joint7']}</param>
                 </state_interface>
             </joint>

Commit message: Mudanca do URDF para usar a malha do link base, ao invés de uma caixa. A malha foi escalada para o tamanho correto e o centro de massa foi ajustado para coincidir com o centro da caixa original. O arquivo STL da malha do link base também foi adicionado ao repositório.

File: src/manip_description/urdf/arm.xacro (robot description, xacro)
@@ -27,7 +27,7 @@
     <visual>
       <geometry>
-        <box size="0.06 0.06 0.10"/>
-      </geometry>
-      <origin xyz="0 0 0.05"/>
+        <mesh filename="package://manip_description/meshes/base_link.stl" scale="0.001 0.001 0.001"/>
+      </geometry>
+      <origin xyz="0 0 0.0"/>
       <material name="red">
         <color rgba="1 0 0 1"/>
@@ -36,11 +36,11 @@
     <collision>
       <geometry>
-        <box size="0.06 0.06 0.10"/>
-      </geometry>
-      <origin xyz="0 0 0.05"/>
+        <mesh filename="package://manip_description/meshes/base_link.stl" scale="0.001 0.001 0.001"/>
+      </geometry>
+      <origin xyz="0 0 0.0"/>
     </collision>
     <inertial>
       <mass value="0.5"/>
-      <origin xyz="0 0 0.05"/>
+      <origin xyz="0 0 0.0"/>
       <inertia ixx="0.0005" ixy="0" ixz="0"
                iyy="0.0005" iyz="0"

Commit message: mudanca no urdf para usar as meshes reais do manipulador

File: src/manip_description/urdf/arm.xacro (robot description, xacro)
@@ -7,15 +7,17 @@
     <visual>
       <geometry>
-        <box size="0.06 0.06 0.02"/>
-      </geometry>
-    </visual>
-    <collision>
-      <geometry>
-        <box size="0.06 0.06 0.02"/>
-      </geometry>
+        <mesh filename="package://manip_description/meshes/Base.stl" scale="0.001 0.001 0.001"/>
+      </geometry>
+      <origin xyz="0 0 0" rpy="1.57 0 0"/>
+    </visual>
+    <collision>
+      <geometry>
+        <mesh filename="package://manip_description/meshes/Base.stl" scale="0.001 0.001 0.001"/>
+      </geometry>
+      <origin xyz="0 0 0" rpy="1.57 0 0"/>
     </collision>
     <inertial>
       <mass value="0.05"/>
-      <origin xyz="0 0 0"/>
+      <origin xyz="0 0 0" rpy="1.57 0 0"/>
       <inertia ixx="1e-05" ixy="0" ixz="0"
                iyy="1e-05" iyz="0"
@@ -27,7 +29,7 @@
     <visual>
       <geometry>
-        <mesh filename="package://manip_description/meshes/base_link.stl" scale="0.001 0.001 0.001"/>
-      </geometry>
-      <origin xyz="0 0 0.0"/>
+        <mesh filename="package://manip_description/meshes/Foguete.stl" scale="0.001 0.001 0.001"/>
+      </geometry>
+      <origin xyz="0 0 0.0" rpy="1.57 0 1.57"/>
       <material name="red">
         <color rgba="1 0 0 1"/>
@@ -36,7 +38,7 @@
     <collision>
       <geometry>
-        <mesh filename="package://manip_description/meshes/base_link.stl" scale="0.001 0.001 0.001"/>
-      </geometry>
-      <origin xyz="0 0 0.0"/>
+        <mesh filename="package://manip_description/meshes/Foguete.stl" scale="0.001 0.001 0.001"/>
+      </geometry>
+      <origin xyz="0 0 0.0" rpy="1.57 0 1.57"/>
     </collision>
     <inertial>
@@ -52,7 +54,7 @@
     <visual>
       <geometry>
-        <box size="0.06 0.06 0.20"/>
-      </geometry>
-      <origin xyz="0 0 0.10"/>
+        <mesh filename="package://manip_description/meshes/Link1.stl" scale="0.001 0.001 0.001"/>
+      </geometry>
+      <origin xyz="0.001 0 -0.012" rpy="1.57 0 3.14"/>
       <material name="green">
         <color rgba="0 1 0 1"/>
@@ -61,11 +63,11 @@
     <collision>
       <geometry>
-        <box size="0.06 0.06 0.20"/>
-      </geometry>
-      <origin xyz="0 0 0.10"/>
+        <mesh filename="package://manip_description/meshes/Link1.stl" scale="0.001 0.001 0.001"/>
+      </geometry>
+      <origin xyz="0.001 0 -0.012" rpy="1.57 0 3.14"/>
     </collision>
     <inertial>
       <mass value="0.4"/>
-      <origin xyz="0 0 0.10"/>
+      <origin xyz="0.001 0 -0.012" rpy="1.57 0 3.14"/>
       <inertia ixx="0.0004" ixy="0" ixz="0"
                iyy="0.0004" iyz="0"
@@ -77,7 +79,7 @@
     <visual>
       <geometry>
-        <box size="0.06 0.06 0.20"/>
-      </geometry>
-      <origin xyz="0 0 0.10"/>
+        <mesh filename="package://manip_description/meshes/Link1.stl" scale="0.001 0.001 0.001"/>
+      </geometry>
+      <origin xyz="0.001 0 -0.011" rpy="1.57 0 3.14"/>
       <material name="blue">
         <color rgba="0 0 1 1"/>
@@ -86,11 +88,11 @@
     <collision>
       <geometry>
-        <box size="0.06 0.06 0.20"/>
-      </geometry>
-      <origin xyz="0 0 0.10"/>
+        <mesh filename="package://manip_description/meshes/Link1.stl" scale="0.001 0.001 0.001"/>
+      </geometry>
+      <origin xyz="0.001 0 -0.0011" rpy="1.57 0 3.14"/>
     </collision>
     <inertial>
       <mass value="0.4"/>
-      <origin xyz="0 0 0.10"/>
+      <origin xyz="0 0 0"/>
       <inertia ixx="0.0004" ixy="0" ixz="0"
                iyy="0.0004" iyz="0"
@@ -102,7 +104,7 @@
     <visual>
       <geometry>
-        <box size="0.06 0.06 0.10"/>
-      </geometry>
-      <origin xyz="0 0 0.05"/>
+        <mesh filename="package://manip_description/meshes/Link3.stl" scale="0.001 0.001 0.001"/>
+      </geometry>
+      <origin xyz="0.042 0 0.020" rpy="1.57 0 1.57"/>
       <material name="yellow">
         <color rgba="1 1 0 1"/>
@@ -111,11 +113,11 @@
     <collision>
       <geometry>
-        <box size="0.06 0.06 0.10"/>
-      </geometry>
-      <origin xyz="0 0 0.05"/>
+        <mesh filename="package://manip_description/meshes/Link3.stl" scale="0.001 0.001 0.001"/>
+      </geometry>
+      <origin xyz="0.042 0 0.020" rpy="1.57 0 1.57"/>
     </collision>
     <inertial>
       <mass value="0.3"/>
-      <origin xyz="0 0 0.05"/>
+      <origin xyz="0.042 0 0.020" rpy="1.57 0 1.57"/>
       <inertia ixx="0.0003" ixy="0" ixz="0"
                iyy="0.0003" iyz="0"
@@ -127,7 +129,7 @@
     <visual>
       <geometry>
-        <box size="0.123 0.0793 0.006"/>
-      </geometry>
-      <origin xyz="0 0 0.003"/>
+        <mesh filename="package://manip_description/meshes/Garra430_teste.stl" scale="0.001 0.001 0.001"/>
+      </geometry>
+      <origin xyz="0.0005 0 -0.004 " rpy="0.0 0 3.14"/>
       <material name="cyan">
         <color rgba="0 1 1 1"/>
@@ -136,11 +138,11 @@
     <collision>
       <geometry>
-        <box size="0.123 0.0793 0.006"/>
-      </geometry>
-      <origin xyz="0 0 0.003"/>
+        <mesh filename="package://manip_description/meshes/Garra430_teste.stl" scale="0.001 0.001 0.001"/>
+      </geometry>
+      <origin xyz="0.0005 0 -0.004" rpy="0.0 0 3.14"/>
     </collision>
     <inertial>
       <mass value="0.15"/>
-      <origin xyz="0 0 0.003"/>
+      <origin xyz="0.0005 0 -0.004" rpy="0.0 0 3.14"/>
       <inertia ixx="7.9e-05" ixy="0" ixz="0"
                iyy="1.9e-04" iyz="0"
@@ -156,5 +158,5 @@
       Ajuste da pose da câmera em relação ao flange
       -->
-      <origin xyz="0 -0.038 0.011"
+      <origin xyz="0 -0.055 0.009"
               rpy="0 -1.57079632679 -1.57079632679"/>
   </xacro:sensor_d455>
@@ -170,5 +172,5 @@
     <parent link="link1"/>
     <child link="link2"/>
-    <origin xyz="0 0 0.10"/>
+    <origin xyz="0 0 0.099"/>
     <axis xyz="0 1 0"/>
     <limit lower="-1.8" upper="1.8"
@@ -178,5 +180,5 @@
     <parent link="link2"/>
     <child link="link3"/>
-    <origin xyz="0 0 0.20"/>
+    <origin xyz="0 0 0.184"/>
     <axis xyz="0 1 0"/>
     <limit lower="-2.6" upper="2.6"
@@ -186,5 +188,5 @@
     <parent link="link3"/>
     <child link="link4"/>
-    <origin xyz="0 0 0.20"/>
+    <origin xyz="0 0 0.185"/>
     <axis xyz="0 1 0"/>
     <limit lower="-2.2" upper="2.2"
@@ -194,5 +196,5 @@
     <parent link="link4"/>
     <child link="link5"/>
-    <origin xyz="0 0 0.10"/>
+    <origin xyz="0.0013 0 0.08"/>
     <axis xyz="0 0 1"/>
     <limit lower="-3.14" upper="3.14"
@@ -212,5 +214,5 @@
     <parent link="link5"/>
     <child link="tcp"/>
-    <origin xyz="0 0 0.15" rpy="0 0 0"/>
+    <origin xyz="0 -0.001 0.16" rpy="0 0 0"/>
   </joint>
   <!-- ==================== TCP 2 ==================-->
@@ -227,5 +229,5 @@
     <parent link="link5"/>
     <child link="tcp2"/>
-    <origin xyz="0 0 0.3" rpy="0 0 0"/>
+    <origin xyz="0 -0.001 0.3" rpy="0 0 0"/>
   </joint>
 </robot>

File: src/manip_description/urdf/gripper.xacro (robot description, xacro)
@@ -4,7 +4,7 @@
     <visual>
         <geometry>
-        <box size="0.123 0.0793 0.00"/>
+        <box size="0.123 0.05 0.00"/>
         </geometry>
-        <origin xyz="0 0 0"/>
+        <origin xyz="0.0013 -0.026 -0.001"/>
         <material name="grey">
         <color rgba="0.6 0.6 0.6 1"/>
@@ -15,7 +15,7 @@
     <visual>
         <geometry>
-        <box size="0.02525 0.02525 0.13425"/>
+        <mesh filename="package://manip_description/meshes/garra.stl" scale="0.0001 0.0001 0.0001"/>
         </geometry>
-        <origin xyz="0 0.025 0.067125"/>
+        <origin xyz="0.024 0.2825 -0.301" rpy="0 3.14 -3.14"/>
         <material name="grey">
         <color rgba="0.6 0.6 0.6 1"/>
@@ -24,11 +24,11 @@
     <collision>
         <geometry>
-        <box size="0.02525 0.02525 0.13425"/>
+        <mesh filename="package://manip_description/meshes/garra.stl" scale="0.0001 0.0001 0.0001"/>
         </geometry>
-        <origin xyz="0 0.025 0.067125"/>
+        <origin xyz="0.024 0.283 -0.301" rpy="0 3.14 -3.14"/>
     </collision>
     <inertial>
         <mass value="0.05"/>
-        <origin xyz="0 0.025 0.067125"/>
+        <origin xyz="0.024 0.283 -0.301" rpy="0 3.14 -3.14"/>
         <inertia ixx="3e-05" ixy="0" ixz="0" iyy="3e-05" iyz="0" izz="8e-06"/>
     </inertial>
@@ -37,5 +37,5 @@
     <parent link="gripper_base_link"/>
     <child link="finger_left"/>
-    <origin xyz="-0.025325 0 0.006"/>
+    <origin xyz="-0.0227 0 0.013"/>
     <axis xyz="0 1 0"/>
     <limit lower="-1.0" upper="1.0" effort="1" velocity="5"/>
@@ -44,18 +44,18 @@
     <visual>
         <geometry>
-        <box size="0.02525 0.02525 0.13425"/>
+        <mesh filename="package://manip_description/meshes/garra.stl" scale="0.0001 0.0001 0.0001"/>
         </geometry>
-        <origin xyz="0 0.025 0.067125"/>
+        <origin xyz="-0.024 -0.283 -0.301" rpy="0 3.14 0"/>
         <material name="grey"/>
     </visual>
     <collision>
         <geometry>
-        <box size="0.02525 0.02525 0.13425"/>
+        <mesh filename="package://manip_description/meshes/garra.stl" scale="0.0001 0.0001 0.0001"/>
         </geometry>
-        <origin xyz="0 0.025 0.067125"/>
+        <origin xyz="-0.024 -0.283 -0.301" rpy="0 3.14 0"/>
     </collision>
     <inertial>
         <mass value="0.05"/>
-        <origin xyz="0 0.025 0.067125"/>
+        <origin xyz="-0.024 -0.283 -0.301" rpy="0 3.14 0"/>
         <inertia ixx="3e-05" ixy="0" ixz="0" iyy="3e-05" iyz="0" izz="8e-06"/>
     </inertial>
@@ -64,5 +64,5 @@
     <parent link="gripper_base_link"/>
     <child link="finger_right"/>
-    <origin xyz="0.025325 0 0.006"/>
+    <origin xyz="0.027 0 0.013"/>
     <axis xyz="0 -1 0"/>
     <limit lower="-1.0" upper="1.0" effort="1" velocity="5"/>
