Commit message: stl arrumado

File: src/manip_description/urdf/arm.xacro (robot description, xacro)
@@ -7,17 +7,17 @@
     <visual>
       <geometry>
-        <mesh filename="package://manip_description/meshes/Base.stl" scale="0.001 0.001 0.001"/>
-      </geometry>
-      <origin xyz="0 0 0" rpy="1.57 0 0"/>
-    </visual>
-    <collision>
-      <geometry>
-        <mesh filename="package://manip_description/meshes/Base.stl" scale="0.001 0.001 0.001"/>
-      </geometry>
-      <origin xyz="0 0 0" rpy="1.57 0 0"/>
+        <mesh filename="package://manip_description/meshes/base_link.stl" scale="0.001 0.001 0.001"/>
+      </geometry>
+      <origin xyz="0 0 0" rpy="0 0 0"/>
+    </visual>
+    <collision>
+      <geometry>
+        <mesh filename="package://manip_description/meshes/base_link.stl" scale="0.001 0.001 0.001"/>
+      </geometry>
+      <origin xyz="0 0 0" rpy="0 0 0"/>
     </collision>
     <inertial>
       <mass value="0.05"/>
-      <origin xyz="0 0 0" rpy="1.57 0 0"/>
+      <origin xyz="0 0 0" rpy="0 0 0"/>
       <inertia ixx="1e-05" ixy="0" ixz="0"
                iyy="1e-05" iyz="0"
@@ -25,11 +25,11 @@
     </inertial>
   </link>
-  <!-- ================= LINK1 ================= -->
+  <!-- ================= LINK1 - FOGUETE ================= -->
   <link name="link1">
     <visual>
       <geometry>
-        <mesh filename="package://manip_description/meshes/Foguete.stl" scale="0.001 0.001 0.001"/>
-      </geometry>
-      <origin xyz="0 0 0.0" rpy="1.57 0 1.57"/>
+        <mesh filename="package://manip_description/meshes/link1.stl" scale="0.001 0.001 0.001"/>
+      </geometry>
+      <origin xyz="0 0 0.0" rpy="0 0 0"/>
       <material name="red">
         <color rgba="1 0 0 1"/>
@@ -38,7 +38,7 @@
     <collision>
       <geometry>
-        <mesh filename="package://manip_description/meshes/Foguete.stl" scale="0.001 0.001 0.001"/>
-      </geometry>
-      <origin xyz="0 0 0.0" rpy="1.57 0 1.57"/>
+        <mesh filename="package://manip_description/meshes/link1.stl" scale="0.001 0.001 0.001"/>
+      </geometry>
+      <origin xyz="0 0 0.0" rpy="0 0 0"/>
     </collision>
     <inertial>
@@ -50,11 +50,11 @@
     </inertial>
   </link>
-  <!-- ================= LINK2 ================= -->
+  <!-- ================= LINK2 - (numero 01)================= -->
   <link name="link2">
     <visual>
       <geometry>
-        <mesh filename="package://manip_description/meshes/Link1.stl" scale="0.001 0.001 0.001"/>
-      </geometry>
-      <origin xyz="0.001 0 -0.012" rpy="1.57 0 3.14"/>
+        <mesh filename="package://manip_description/meshes/link2.stl" scale="0.001 0.001 0.001"/>
+      </geometry>
+      <origin xyz="0 0 -0.09775" rpy="0 0 0"/>
       <material name="green">
         <color rgba="0 1 0 1"/>
@@ -63,11 +63,11 @@
     <collision>
       <geometry>
-        <mesh filename="package://manip_description/meshes/Link1.stl" scale="0.001 0.001 0.001"/>
-      </geometry>
-      <origin xyz="0.001 0 -0.012" rpy="1.57 0 3.14"/>
+        <mesh filename="package://manip_description/meshes/link2.stl" scale="0.001 0.001 0.001"/>
+      </geometry>
+      <origin xyz="0 0 -0.09775" rpy="0 0 0"/>
     </collision>
     <inertial>
       <mass value="0.4"/>
-      <origin xyz="0.001 0 -0.012" rpy="1.57 0 3.14"/>
+      <origin xyz="0 0 -0.09775" rpy="0 0 0"/>
       <inertia ixx="0.0004" ixy="0" ixz="0"
                iyy="0.0004" iyz="0"
@@ -79,7 +79,7 @@
     <visual>
       <geometry>
-        <mesh filename="package://manip_description/meshes/Link1.stl" scale="0.001 0.001 0.001"/>
-      </geometry>
-      <origin xyz="0.001 0 -0.011" rpy="1.57 0 3.14"/>
+        <mesh filename="package://manip_description/meshes/link3.stl" scale="0.001 0.001 0.001"/>
+      </geometry>
+      <origin xyz="0 0 -0.28275" rpy="0 0 0"/>
       <material name="blue">
         <color rgba="0 0 1 1"/>
@@ -88,11 +88,11 @@
     <collision>
       <geometry>
-        <mesh filename="package://manip_description/meshes/Link1.stl" scale="0.001 0.001 0.001"/>
-      </geometry>
-      <origin xyz="0.001 0 -0.0011" rpy="1.57 0 3.14"/>
+        <mesh filename="package://manip_description/meshes/link3.stl" scale="0.001 0.001 0.001"/>
+      </geometry>
+      <origin xyz="0 0 -0.28275" rpy="0 0 0"/>
     </collision>
     <inertial>
       <mass value="0.4"/>
-      <origin xyz="0 0 0"/>
+      <origin xyz="0 0 -0.28275" rpy="0 0 0"/>
       <inertia ixx="0.0004" ixy="0" ixz="0"
                iyy="0.0004" iyz="0"
@@ -104,20 +104,20 @@
     <visual>
       <geometry>
-        <mesh filename="package://manip_description/meshes/Link3.stl" scale="0.001 0.001 0.001"/>
-      </geometry>
-      <origin xyz="0.042 0 0.020" rpy="1.57 0 1.57"/>
+        <mesh filename="package://manip_description/meshes/link4.stl" scale="0.001 0.001 0.001"/>
+      </geometry>
+      <origin xyz="0 0 -0.48775" rpy="0 0 0"/>
       <material name="yellow">
         <color rgba="1 1 0 1"/>
       </material>
-    </visual>
-    <collision>
-      <geometry>
-        <mesh filename="package://manip_description/meshes/Link3.stl" scale="0.001 0.001 0.001"/>
-      </geometry>
-      <origin xyz="0.042 0 0.020" rpy="1.57 0 1.57"/>
+    </visual>link5
+    <collision>
+      <geometry>
+        <mesh filename="package://manip_description/meshes/link4.stl" scale="0.001 0.001 0.001"/>
+      </geometry>
+      <origin xyz="0 0 -0.48775" rpy="0 0 0"/>
     </collision>
     <inertial>
       <mass value="0.3"/>
-      <origin xyz="0.042 0 0.020" rpy="1.57 0 1.57"/>
+      <origin xyz="0 0 -0.48775" rpy="0 0 0"/>
       <inertia ixx="0.0003" ixy="0" ixz="0"
                iyy="0.0003" iyz="0"
@@ -129,7 +129,7 @@
     <visual>
       <geometry>
-        <mesh filename="package://manip_description/meshes/Garra430_teste.stl" scale="0.001 0.001 0.001"/>
-      </geometry>
-      <origin xyz="0.0005 0 -0.004 " rpy="0.0 0 3.14"/>
+        <mesh filename="package://manip_description/meshes/link5.stl" scale="0.001 0.001 0.001"/>
+      </geometry>
+      <origin xyz="0 0 -0.5659" rpy="0.0 0 0"/>
       <material name="cyan">
         <color rgba="0 1 1 1"/>
@@ -138,11 +138,11 @@
     <collision>
       <geometry>
-        <mesh filename="package://manip_description/meshes/Garra430_teste.stl" scale="0.001 0.001 0.001"/>
-      </geometry>
-      <origin xyz="0.0005 0 -0.004" rpy="0.0 0 3.14"/>
+        <mesh filename="package://manip_description/meshes/link5.stl" scale="0.001 0.001 0.001"/>
+      </geometry>
+      <origin xyz="0 0 -0.5659" rpy="0.0 0 0"/>
     </collision>
     <inertial>
       <mass value="0.15"/>
-      <origin xyz="0.0005 0 -0.004" rpy="0.0 0 3.14"/>
+      <origin xyz="0 0 -0.5659" rpy="0.0 0 0"/>
       <inertia ixx="7.9e-05" ixy="0" ixz="0"
                iyy="1.9e-04" iyz="0"
@@ -158,5 +158,5 @@
       Ajuste da pose da câmera em relação ao flange
       -->
-      <origin xyz="0 -0.055 0.009"
+      <origin xyz="0 -0.055 0.0125"
               rpy="0 -1.57079632679 -1.57079632679"/>
   </xacro:sensor_d455>
@@ -172,5 +172,5 @@
     <parent link="link1"/>
     <child link="link2"/>
-    <origin xyz="0 0 0.099"/>
+    <origin xyz="0 0 0.09775"/>
     <axis xyz="0 1 0"/>
     <limit lower="-1.8" upper="1.8"
@@ -180,5 +180,5 @@
     <parent link="link2"/>
     <child link="link3"/>
-    <origin xyz="0 0 0.184"/>
+    <origin xyz="0 0 0.185"/>
     <axis xyz="0 1 0"/>
     <limit lower="-2.6" upper="2.6"
@@ -188,5 +188,5 @@
     <parent link="link3"/>
     <child link="link4"/>
-    <origin xyz="0 0 0.185"/>
+    <origin xyz="0 0 0.205"/>
     <axis xyz="0 1 0"/>
     <limit lower="-2.2" upper="2.2"
@@ -196,5 +196,5 @@
     <parent link="link4"/>
     <child link="link5"/>
-    <origin xyz="0.0013 0 0.08"/>
+    <origin xyz="0 0 0.07815"/>
     <axis xyz="0 0 1"/>
     <limit lower="-3.14" upper="3.14"
@@ -214,5 +214,5 @@
     <parent link="link5"/>
     <child link="tcp"/>
-    <origin xyz="0 -0.001 0.16" rpy="0 0 0"/>
+    <origin xyz="0 0 0.13" rpy="0 0 0"/>
   </joint>
   <!-- ==================== TCP 2 ==================-->
@@ -229,5 +229,5 @@
     <parent link="link5"/>
     <child link="tcp2"/>
-    <origin xyz="0 -0.001 0.3" rpy="0 0 0"/>
+    <origin xyz="0 0 0.3" rpy="0 0 0"/>
   </joint>
 </robot>

File: src/manip_description/urdf/gripper.xacro (robot description, xacro)
@@ -4,7 +4,7 @@
     <visual>
         <geometry>
-        <box size="0.123 0.05 0.00"/>
+        <box size="0.123 0.03 0.00"/>
         </geometry>
-        <origin xyz="0.0013 -0.026 -0.001"/>
+        <origin xyz="0 0 0.00425"/>
         <material name="grey">
         <color rgba="0.6 0.6 0.6 1"/>
@@ -15,7 +15,7 @@
     <visual>
         <geometry>
-        <mesh filename="package://manip_description/meshes/garra.stl" scale="0.0001 0.0001 0.0001"/>
+        <mesh filename="package://manip_description/meshes/left_finger.stl" scale="0.001 0.001 0.001"/>
         </geometry>
-        <origin xyz="0.024 0.2825 -0.301" rpy="0 3.14 -3.14"/>
+        <origin xyz="-0.0252 0 -0.58444" rpy="0 0 0"/>
         <material name="grey">
         <color rgba="0.6 0.6 0.6 1"/>
@@ -24,11 +24,11 @@
     <collision>
         <geometry>
-        <mesh filename="package://manip_description/meshes/garra.stl" scale="0.0001 0.0001 0.0001"/>
+        <mesh filename="package://manip_description/meshes/left_finger.stl" scale="0.001 0.001 0.001"/>
         </geometry>
-        <origin xyz="0.024 0.283 -0.301" rpy="0 3.14 -3.14"/>
+        <origin xyz="-0.0252 0 -0.58444" rpy="0 0 0"/>
     </collision>
     <inertial>
         <mass value="0.05"/>
-        <origin xyz="0.024 0.283 -0.301" rpy="0 3.14 -3.14"/>
+        <origin xyz="-0.0252 0 -0.58444" rpy="0 0 0"/>
         <inertia ixx="3e-05" ixy="0" ixz="0" iyy="3e-05" iyz="0" izz="8e-06"/>
     </inertial>
@@ -37,5 +37,5 @@
     <parent link="gripper_base_link"/>
     <child link="finger_left"/>
-    <origin xyz="-0.0227 0 0.013"/>
+    <origin xyz="-0.0252 0 0.0215"/>
     <axis xyz="0 1 0"/>
     <limit lower="-1.0" upper="1.0" effort="1" velocity="5"/>
@@ -44,18 +44,18 @@
     <visual>
         <geometry>
-        <mesh filename="package://manip_description/meshes/garra.stl" scale="0.0001 0.0001 0.0001"/>
+        <mesh filename="package://manip_description/meshes/right_finger.stl" scale="0.001 0.001 0.001"/>
         </geometry>
-        <origin xyz="-0.024 -0.283 -0.301" rpy="0 3.14 0"/>
+        <origin xyz="0.0252 0 -0.58444" rpy="0 0 0"/>
         <material name="grey"/>
     </visual>
     <collision>
         <geometry>
-        <mesh filename="package://manip_description/meshes/garra.stl" scale="0.0001 0.0001 0.0001"/>
+        <mesh filename="package://manip_description/meshes/right_finger.stl" scale="0.001 0.001 0.001"/>
         </geometry>
-        <origin xyz="-0.024 -0.283 -0.301" rpy="0 3.14 0"/>
+        <origin xyz="0.0252 0 -0.58444" rpy="0 0 0"/>
     </collision>
     <inertial>
         <mass value="0.05"/>
-        <origin xyz="-0.024 -0.283 -0.301" rpy="0 3.14 0"/>
+        <origin xyz="0.0252 0 -0.58444" rpy="0 0 0"/>
         <inertia ixx="3e-05" ixy="0" ixz="0" iyy="3e-05" iyz="0" izz="8e-06"/>
     </inertial>
@@ -64,5 +64,5 @@
     <parent link="gripper_base_link"/>
     <child link="finger_right"/>
-    <origin xyz="0.027 0 0.013"/>
+    <origin xyz="0.0252 0 0.0215"/>
     <axis xyz="0 -1 0"/>
     <limit lower="-1.0" upper="1.0" effort="1" velocity="5"/>

Commit message: adicionado o manipulador para funcionar na raspberry pi

File: src/manip_description/urdf/arm.xacro (robot description, xacro)
@@ -2,5 +2,8 @@
 <robot name="manip" xmlns:xacro="http://ros.org/wiki/xacro">
   <!-- ================= REALSENSE INCLUDE ================= -->
-  <xacro:include filename="$(find realsense2_description)/urdf/_d455.urdf.xacro"/>
+  <xacro:arg name="use_realsense" default="true"/>
+  <xacro:if value="$(arg use_realsense)">
+    <xacro:include filename="$(find realsense2_description)/urdf/_d455.urdf.xacro"/>
+  </xacro:if>
   <!-- ================= BASE ================= -->
   <link name="base_link">
@@ -106,9 +109,9 @@
         <mesh filename="package://manip_description/meshes/link4.stl" scale="0.001 0.001 0.001"/>
       </geometry>
-      <origin xyz="0 0 -0.48775" rpy="0 0 0"/>
+      <origin xyz="0 0 -0.48775" rpy="0 0 3.14"/>
       <material name="yellow">
         <color rgba="1 1 0 1"/>
       </material>
-    </visual>link5
+    </visual>
     <collision>
       <geometry>
@@ -151,14 +154,16 @@
   </link>
   <!-- ================= REALSENSE D455 ================= -->
-  <xacro:sensor_d455
-      parent="link5"
-      name="camera"
-      use_nominal_extrinsics="true">
-      <!--
-      Ajuste da pose da câmera em relação ao flange
-      -->
-      <origin xyz="0 -0.055 0.0125"
-              rpy="0 -1.57079632679 -1.57079632679"/>
-  </xacro:sensor_d455>
+  <xacro:if value="$(arg use_realsense)">
+    <xacro:sensor_d455
+        parent="link5"
+        name="camera"
+        use_nominal_extrinsics="true">
+        <!--
+        Ajuste da pose da câmera em relação ao flange
+        -->
+        <origin xyz="0 -0.055 0.0125"
+                rpy="0 -1.57079632679 -1.57079632679"/>
+    </xacro:sensor_d455>
+  </xacro:if>
   <!-- ================= ARM JOINTS ================= -->
   <joint name="manip_joint1" type="revolute">
@@ -196,5 +201,5 @@
     <parent link="link4"/>
     <child link="link5"/>
-    <origin xyz="0 0 0.07815"/>
+    <origin xyz="-0.03 0 0.07815"/>
     <axis xyz="0 0 1"/>
     <limit lower="-3.14" upper="3.14"
@@ -214,5 +219,5 @@
     <parent link="link5"/>
     <child link="tcp"/>
-    <origin xyz="0 0 0.13" rpy="0 0 0"/>
+    <origin xyz="0 0 0.17" rpy="0 0 0"/>
   </joint>
   <!-- ==================== TCP 2 ==================-->
